Commit message: create gazebo simulation

File: description/robot_core.xacro (robot description, xacro)
@@ -41,4 +41,7 @@
         </xacro:inertial_box>
     </link>
+    <gazebo reference = "chassis">
+        <material>Gazebo/White</material>
+    </gazebo>
     <!-- Left Wheel Link -->
     <link name = "left_wheel">
@@ -58,4 +61,7 @@
         </xacro:inertial_cylinder>
     </link>
+    <gazebo reference = "left_wheel">
+        <material>Gazebo/Blue</material>
+    </gazebo>
     <!-- Right Wheel Link -->
     <link name = "right_wheel">
@@ -75,4 +81,7 @@
         </xacro:inertial_cylinder>
     </link>
+    <gazebo reference = "right_wheel">
+        <material>Gazebo/Blue</material>
+    </gazebo>
    <!-- Caster Wheel Link -->
     <link name = "caster_wheel">
@@ -92,4 +101,9 @@
         </xacro:inertial_sphere>
     </link>
+    <gazebo reference = "caster_wheel">
+        <material>Gazebo/Black</material>
+        <mu1 value = "0.001" />
+        <mu2 value = "0.001" />
+    </gazebo>
 <!-- Joints -->
     <!-- Chassis Joint -->

Commit message: slam mapping

File: description/robot_core.xacro (robot description, xacro)
@@ -21,4 +21,7 @@
     <!-- Base Link -->
     <link name = "base_link">
+    </link>
+    <!-- Base Footprint Link -->
+    <link name = "base_footprint">
     </link>
     <!-- Chassis Link -->
@@ -107,4 +110,10 @@
     </gazebo>
 <!-- Joints -->
+    <!-- Base Footprint Joint -->
+    <joint name = "base_footprint_joint" type = "fixed">
+        <parent link = "base_link"/>
+        <child link = "base_footprint"/>
+        <origin xyz = "0 0 0" rpy = "0 0 0"/>
+    </joint>
     <!-- Chassis Joint -->
     <joint name = "chassis_joint" type = "fixed">
